File: MotorDriverV1_0.kicad_pcb (KiCad board)
At the start: 2 copper layers, 68.6 x 53.3 mm, 44 parts, among them J1 Screw_Terminal_01x02, J10 Conn_01x02, J11 Conn_01x02, J12 Conn_01x02, J2 Conn_01x02, J3 Conn_01x02, J4 Conn_01x02, J5 Screw_Terminal_01x02, J6 Screw_Terminal_01x02, J7 Conn_01x02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

Commit message: some routing and compoment placement
Parts:
- added J13: Conn_01x01, Connector_PinHeader_2.54mm:PinHeader_1x01_P2.54mm_Vertical, F.Cu at (141.5, 109.9)
- J10: value Conn_01x02 -> Conn_02x06_Odd_Even; footprint Connector_PinHeader_2.54mm:PinHeader_1x02_P2.54mm_Vertical -> Connector_IDC:IDC-Header_2x06_P2.54mm_Vertical
- J11, J12, J7, J8, J9: value Conn_01x02 -> Conn_01x01; footprint Connector_PinHeader_2.54mm:PinHeader_1x02_P2.54mm_Vertical -> Connector_PinHeader_2.54mm:PinHeader_1x01_P2.54mm_Vertical
- moved J3 189.0 mm to (178.3, 101.0), turned to 180 degrees
- moved J4 158.1 mm to (155.4, 84.5)
- moved J7 149.0 mm to (128.8, 117.5)
- moved J8 148.2 mm to (131.3, 117.5)
- moved J9 143.8 mm to (133.9, 117.5)
- moved J2 143.8 mm to (119.9, 106.0)
- moved J12 137.4 mm to (138.9, 109.9)
- moved J10 136.5 mm to (128.8, 114.9), turned to 90 degrees
- moved J11 134.6 mm to (136.4, 109.9)
- moved R5 131.3 mm to (178.3, 114.9), turned to 90 degrees
- moved C5 126.8 mm to (174.5, 116.2), turned to 90 degrees
- moved D3 107.6 mm to (174.5, 87.0)
- moved D1 102.4 mm to (174.5, 81.9)
- moved D2 101.9 mm to (174.5, 79.4)
- moved C6 101.5 mm to (150.4, 111.1), turned to 270 degrees
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Connections:
- J10 pad 1: /CSEN2 -> /TF1
- J10 pad 2: /A1 -> GND
- J11 pad 1: /TF2 -> /8
- J12 pad 1: /TF1 -> /A1
- J7 pad 1: /BR2 -> /7
- J8 pad 1: /BR1 -> /A0
- J9 pad 1: /CSEN1 -> /6(**)
- P1 pad 1: Net-(P1-Pad1) -> (no net)
- P1 pad 2: /IOREF -> (no net)
- P1 pad 3: /Reset -> (no net)
- P1 pad 4: +3V3 -> (no net)
- P2 pad 3: /A2 -> (no net)
- P2 pad 4: /A3 -> (no net)
- P3 pad 3: /AREF -> (no net)
- P3 pad 5: /13(SCK) -> (no net)
- P3 pad 6: /12(MISO) -> (no net)
- P3 pad 7: /11(**/MOSI) -> (no net)
- P3 pad 8: /10(**/SS) -> (no net)
- P4 pad 7: /1(Tx) -> (no net)
- P4 pad 8: /0(Rx) -> (no net)
- P5 pad 1: Net-(P5-Pad1) -> (no net)
- P6 pad 1: Net-(P6-Pad1) -> (no net)
- P7 pad 1: Net-(P7-Pad1) -> (no net)
- P8 pad 1: Net-(P8-Pad1) -> (no net)
Routing:
- net GND: track 0.00 -> 258.4 mm, vias 0 -> 6
- net /Vs: track 0.00 -> 129.9 mm, vias 0 -> 2
- net Net-(C5-Pad1): track 0.00 -> 62.1 mm
- net /Vin: track 0.00 -> 59.6 mm, vias 0 -> 2
- net Net-(C6-Pad2): track 0.00 -> 53.5 mm
- net Net-(C8-Pad2): track 0.00 -> 48.6 mm
- net /BR2: track 0.00 -> 24.0 mm, vias 0 -> 2
- net /CSEN1: track 0.00 -> 21.2 mm
- net Net-(D3-Pad2): track 0.00 -> 19.5 mm
- net Net-(D2-Pad2): track 0.00 -> 19.2 mm
- net Net-(C7-Pad1): track 0.00 -> 17.8 mm
- net Net-(D4-Pad2): track 0.00 -> 11.6 mm, vias 0 -> 2
- net Net-(D1-Pad2): track 0.00 -> 11.6 mm, vias 0 -> 2
- net /CSEN2: track 0.00 -> 8.23 mm, vias 0 -> 1
- net Net-(C2-Pad1): track 0.00 -> 5.08 mm
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Other:
- net class Power added: clearance 0.2, trace_width 0.25, via_dia 0.6, via_drill 0.4

Commit message: routing completed
Connections:
- P2 pad 5: /A4(SDA) -> (no net)
- P2 pad 6: /A5(SCL) -> (no net)
- P3 pad 1: /A5(SCL) -> (no net)
- P3 pad 2: /A4(SDA) -> (no net)
Routing:
- net +5V: track 0.00 -> 88.6 mm, vias 0 -> 3
- net /2: track 0.00 -> 79.1 mm, vias 0 -> 2
- net /6(**): track 0.00 -> 70.7 mm, vias 0 -> 3
- net /4: track 0.00 -> 69.9 mm, vias 0 -> 3
- net /5(**): track 0.00 -> 65.7 mm, vias 0 -> 4
- net /7: track 0.00 -> 64.8 mm, vias 0 -> 2
- net /3(**): track 0.00 -> 64.0 mm, vias 0 -> 4
- net /BR1: track 0.00 -> 57.5 mm, vias 0 -> 3
- net /8: track 0.00 -> 46.6 mm
- net /9(**): track 0.00 -> 38.0 mm
- net /A1: track 0.00 -> 36.6 mm
- net /TF1: track 0.00 -> 36.0 mm
- net /A0: track 0.00 -> 34.9 mm
- net /CSEN1: track 21.2 -> 54.0 mm, vias 0 -> 1
- net /CSEN2: track 8.23 -> 40.0 mm
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