File: MotorDriverV1_0.sch (KiCad schematic (older format))
At the start: 44 parts, among them J1 Screw_Terminal_01x02, J10 Conn_01x02, J11 Conn_01x02, J12 Conn_01x02, J2 Conn_01x02, J3 Conn_01x02, J4 Conn_01x02, J5 Screw_Terminal_01x02, J6 Screw_Terminal_01x02, J7 Conn_01x02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

Commit message: some routing and compoment placement
Parts:
- removed J10, J11, J12, J7, J8, J9: Conn_01x02, Connector_PinHeader_2.54mm:PinHeader_1x02_P2.54mm_Vertical, symbol Connector_Generic:Conn_01x02
- added J10: Conn_02x06_Odd_Even, Connector_IDC:IDC-Header_2x06_P2.54mm_Vertical, symbol Connector_Generic:Conn_02x06_Odd_Even
- added J11, J12, J13, J7, J8, J9: Conn_01x01, Connector_PinHeader_2.54mm:PinHeader_1x01_P2.54mm_Vertical, symbol Connector_Generic:Conn_01x01
Connections:
- wire segments 106 -> 115
Other:
- note added: "BR1 -- 6(**)\nCSEN1 -- A0\nTF1 -- 7\n\nBR2 -- 8\nCSEN2 -- A1\nTF2 -- 9(**)\n\npositionne de facon a mettre un jumper en configuration shield\n"
Changed lines of the file:
@@
 	1    0    0    -1
 $EndComp
-Text Label 9000 4750 0    60   ~ 0
+Text Label 9250 5000 0    60   ~ 0
 2
-Text Label 9000 4650 0    60   ~ 0
+Text Label 8700 5100 0    60   ~ 0
 3(**)
-Text Label 9000 4550 0    60   ~ 0
+Text Label 11050 4900 0    60   ~ 0
 4
-Text Label 9000 4450 0    60   ~ 0
+Text Label 10750 4800 0    60   ~ 0
 5(**)
 Wire Wire Line
-	8650 4750 9000 4750
-Wire Wire Line
-	8650 4550 9000 4550
-Wire Wire Line
-	8650 4450 9000 4450
-Wire Wire Line
-	8650 4350 9000 4350
-Wire Wire Line
-	8650 4000 9000 4000
-$Comp
-L Connector_Generic:Conn_01x02 J7
-U 1 1 5C1F806C
-P 8550 3800
-F 0 "J7" V 8516 3612 50  0000 R CNN
-F 1 "Conn_01x02" V 8425 3612 50  0000 R CNN
-F 2 "Connector_PinHeader_2.54mm:PinHeader_1x02_P2.54mm_Vertical" H 8550 3800 50  0001 C CNN
-F 3 "~" H 8550 3800 50  0001 C CNN
-	1    8550 3800
-	0    -1   -1   0
-$EndComp
-$Comp
-L Connector_Generic:Conn_01x02 J8
-U 1 1 5C1F81B3
-P 8550 4150
-F 0 "J8" V 8516 3962 50  0000 R CNN
-F 1 "Conn_01x02" V 8425 3962 50  0000 R CNN
-F 2 "Connector_PinHeader_2.54mm:PinHeader_1x02_P2.54mm_Vertical" H 8550 4150 50  0001 C CNN
-F 3 "~" H 8550 4150 50  0001 C CNN
-	1    8550 4150
-	0    -1   -1   0
-$EndComp
-Text Label 8550 4000 2    50   ~ 0
-BR2
-Text Label 8550 4350 2    50   ~ 0
-BR1
-Text Label 9000 5100 0    60   ~ 0
-A0
-Text Label 9000 5450 0    60   ~ 0
-A1
-Text Label 8650 4450 0    50   ~ 0
+	8900 5000 9100 5000
+Wire Wire Line
+	10700 4900 10900 4900
+Wire Wire Line
+	10400 4800 10650 4800
+Text Label 10400 4800 0    50   ~ 0
 PWM2
 Wire Wire Line
-	8650 4650 9000 4650
-Text Label 8650 4650 0    50   ~ 0
+	8350 5100 8550 5100
+Text Label 8350 5100 0    50   ~ 0
 PWM1
-Text Label 8650 4550 0    50   ~ 0
+Text Label 10700 4900 0    50   ~ 0
 DIR2
-Text Label 8650 4750 0    50   ~ 0
+Text Label 8900 5000 0    50   ~ 0
 DIR1
-Text Label 9000 4350 0    50   ~ 0
-7
-Text Label 9000 4000 0    50   ~ 0
-8
-$Comp
-L Connector_Generic:Conn_01x02 J9
-U 1 1 5C2152B0
-P 8550 4900
-F 0 "J9" V 8516 4712 50  0000 R CNN
-F 1 "Conn_01x02" V 8425 4712 50  0000 R CNN
-F 2 "Connector_PinHeader_2.54mm:PinHeader_1x02_P2.54mm_Vertical" H 8550 4900 50  0001 C CNN
-F 3 "~" H 8550 4900 50  0001 C CNN
-	1    8550 4900
-	0    -1   -1   0
-$EndComp
-$Comp
-L Connector_Generic:Conn_01x02 J10
-U 1 1 5C215407
-P 8550 5250
-F 0 "J10" V 8516 5062 50  0000 R CNN
-F 1 "Conn_01x02" V 8425 5062 50  0000 R CNN
-F 2 "Connector_PinHeader_2.54mm:PinHeader_1x02_P2.54mm_Vertical" H 8550 5250 50  0001 C CNN
-F 3 "~" H 8550 5250 50  0001 C CNN
-	1    8550 5250
-	0    -1   -1   0
-$EndComp
-Wire Wire Line
-	8650 5450 9000 5450
-Wire Wire Line
-	8650 5100 9000 5100
-Text Label 8550 5100 2    50   ~ 0
-CSEN1
-Text Label 8550 5450 2    50   ~ 0
-CSEN2
-Text Label 9000 6150 0    60   ~ 0
-6(**)
-Text Label 9000 5800 0    60   ~ 0
-9(**)
-Wire Wire Line
-	8650 5800 9000 5800
-Wire Wire Line
-	8650 6150 9000 6150
-$Comp
-L Connector_Generic:Conn_01x02 J11
-U 1 1 5C22C9E4
-P 8550 5600
-F 0 "J11" V 8516 5412 50  0000 R CNN
-F 1 "Conn_01x02" V 8425 5412 50  0000 R CNN
-F 2 "Connector_PinHeader_2.54mm:PinHeader_1x02_P2.54mm_Vertical" H 8550 5600 50  0001 C CNN
-F 3 "~" H 8550 5600 50  0001 C CNN
-	1    8550 5600
-	0    -1   -1   0
-$EndComp
-$Comp
-L Connector_Generic:Conn_01x02 J12
-U 1 1 5C22CB03
-P 8550 5950
-F 0 "J12" V 8516 5762 50  0000 R CNN
-F 1 "Conn_01x02" V 8425 5762 50  0000 R CNN
-F 2 "Connector_PinHeader_2.54mm:PinHeader_1x02_P2.54mm_Vertical" H 8550 5950 50  0001 C CNN
-F 3 "~" H 8550 5950 50  0001 C CNN
-	1    8550 5950
-	0    -1   -1   0
-$EndComp
-Text Label 8550 5800 2    50   ~ 0
-TF2
-Text Label 8550 6150 2    50   ~ 0
-TF1
 $Comp
 L Driver_Motor:LMD18200 U4
@@
 Text Label 2050 6300 0    50   ~ 0
 GND
+$Comp
+L Connector_Generic:Conn_02x06_Odd_Even J10
+U 1 1 5C508C2B
+P 9800 5000
+F 0 "J10" H 9850 5417 50  0000 C CNN
+F 1 "Conn_02x06_Odd_Even" H 9850 5326 50  0000 C CNN
+F 2 "Connector_IDC:IDC-Header_2x06_P2.54mm_Vertical" H 9800 5000 50  0001 C CNN
+F 3 "~" H 9800 5000 50  0001 C CNN
+	1    9800 5000
+	1    0    0    -1
+$EndComp
+Text Label 10100 4800 0    50   ~ 0
+GND
+Text Label 9600 5300 2    50   ~ 0
+GND
+Wire Wire Line
+	10100 4900 10650 4900
+Wire Wire Line
+	10650 4900 10650 4800
+Connection ~ 10650 4800
+Wire Wire Line
+	10650 4800 10750 4800
+Wire Wire Line
+	10100 5000 10900 5000
+Wire Wire Line
+	10900 5000 10900 4900
+Connection ~ 10900 4900
+Wire Wire Line
+	10900 4900 11050 4900
+$Comp
+L Connector_Generic:Conn_01x01 J11
+U 1 1 5C524EA5
+P 9800 5850
+F 0 "J11" H 9720 5625 50  0000 C CNN
+F 1 "Conn_01x01" H 9720 5716 50  0000 C CNN
+F 2 "Connector_PinHeader_2.54mm:PinHeader_1x01_P2.54mm_Vertical" H 9800 5850 50  0001 C CNN
+F 3 "~" H 9800 5850 50  0001 C CNN
+	1    9800 5850
+	-1   0    0    1
+$EndComp
+Text Label 10250 5850 0    50   ~ 0
+8
+$Comp
+L Connector_Generic:Conn_01x01 J12
+U 1 1 5C525119
+P 9800 5950
+F 0 "J12" H 9720 5725 50  0000 C CNN
+F 1 "Conn_01x01" H 9720 5816 50  0000 C CNN
+F 2 "Connector_PinHeader_2.54mm:PinHeader_1x01_P2.54mm_Vertical" H 9800 5950 50  0001 C CNN
+F 3 "~" H 9800 5950 50  0001 C CNN
+	1    9800 5950
+	-1   0    0    1
+$EndComp
+$Comp
+L Connector_Generic:Conn_01x01 J13
+U 1 1 5C525330
+P 9800 6050
+F 0 "J13" H 9720 5825 50  0000 C CNN
+F 1 "Conn_01x01" H 9720 5916 50  0000 C CNN
+F 2 "Connector_PinHeader_2.54mm:PinHeader_1x01_P2.54mm_Vertical" H 9800 6050 50  0001 C CNN
+F 3 "~" H 9800 6050 50  0001 C CNN
+	1    9800 6050
+	-1   0    0    1
+$EndComp
+$Comp
+L Connector_Generic:Conn_01x01 J7
+U 1 1 5C525452
+P 9750 4100
+F 0 "J7" H 9830 4142 50  0000 L CNN
+F 1 "Conn_01x01" H 9830 4051 50  0000 L CNN
+F 2 "Connector_PinHeader_2.54mm:PinHeader_1x01_P2.54mm_Vertical" H 9750 4100 50  0001 C CNN
+F 3 "~" H 9750 4100 50  0001 C CNN
+	1    9750 4100
+	1    0    0    -1
+$EndComp
+$Comp
+L Connector_Generic:Conn_01x01 J8
+U 1 1 5C52552F
+P 9750 4200
+F 0 "J8" H 9830 4242 50  0000 L CNN
+F 1 "Conn_01x01" H 9830 4151 50  0000 L CNN
+F 2 "Connector_PinHeader_2.54mm:PinHeader_1x01_P2.54mm_Vertical" H 9750 4200 50  0001 C CNN
+F 3 "~" H 9750 4200 50  0001 C CNN
+	1    9750 4200
+	1    0    0    -1
+$EndComp
+$Comp
+L Connector_Generic:Conn_01x01 J9
+U 1 1 5C5255CB
+P 9750 4300
+F 0 "J9" H 9830 4342 50  0000 L CNN
+F 1 "Conn_01x01" H 9830 4251 50  0000 L CNN
+F 2 "Connector_PinHeader_2.54mm:PinHeader_1x01_P2.54mm_Vertical" H 9750 4300 50  0001 C CNN
+F 3 "~" H 9750 4300 50  0001 C CNN
+	1    9750 4300
+	1    0    0    -1
+$EndComp
+Wire Wire Line
+	10250 5850 10000 5850
+Text Label 10250 5950 0    50   ~ 0
+A1
+Text Label 10250 6050 0    50   ~ 0
+9(**)
+Wire Wire Line
+	10250 5950 10000 5950
+Wire Wire Line
+	10000 6050 10250 6050
+Text Label 10100 5100 0    50   ~ 0
+BR2
+Text Label 10100 5200 0    50   ~ 0
+CSEN2
+Text Label 10100 5300 0    50   ~ 0
+TF2
+Text Notes 8000 7000 0    50   ~ 0
+BR1 -- 6(**)\nCSEN1 -- A0\nTF1 -- 7\n\nBR2 -- 8\nCSEN2 -- A1\nTF2 -- 9(**)\n\npositionne de facon a mettre un jumper en configuration shield\n
+Text Label 9600 4800 2    50   ~ 0
+TF1
+Text Label 9600 4900 2    50   ~ 0
+CSEN1
+Text Label 9600 5000 2    50   ~ 0
+BR1
+Wire Wire Line
+	9100 5000 9100 5100
+Wire Wire Line
+	9100 5100 9600 5100
+Connection ~ 9100 5000
+Wire Wire Line
+	9100 5000 9250 5000
+Wire Wire Line
+	9600 5200 8550 5200
+Wire Wire Line
+	8550 5200 8550 5100
+Connection ~ 8550 5100
+Wire Wire Line
+	8550 5100 8700 5100
+Text Label 9550 4100 0    50   ~ 0
+7
+Text Label 9550 4200 0    50   ~ 0
+A0
+Text Label 9550 4300 0    50   ~ 0
+6(**)
 $EndSCHEMATC

Commit message: routing completed
Connections:
- net labels added: A4(SDA_2), A5(SCL_2)
Changed lines of the file:
@@
 A3
 Text Label 8900 2900 0    60   ~ 0
-A4(SDA)
+A4(SDA_2)
 Text Label 8900 3000 0    60   ~ 0
-A5(SCL)
+A5(SCL_2)
 Text Label 10550 3000 0    60   ~ 0
 0(Rx)
